File: pcb/hackpad.kicad_pcb (KiCad board)
At the start: 2 copper layers, 19.4 x 76.2 mm, 5 parts, among them SW1 SW_Push, SW2 SW_Push, SW3 SW_Push, SW4 RotaryEncoder_Switch, U1 MOUDLE-SEEEDUINO-XIAO

Commit message: NewChanges
Routing:
- net Net-(U1-PB08_A6_D6_TX): track 57.4 -> 113.3 mm
- net GND: track 115.6 -> 152.7 mm
- net Net-(U1-PA9_A5_D5_SCL): track 43.9 -> 78.7 mm
- net Net-(U1-PB09_A7_D7_RX): track 34.6 -> 44.2 mm
Changed lines of the file:
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@@
+	)
+	(segment
+		(start 111.43 137.1)
+		(end 115.12 133.41)
+		(width 0.2)
+		(layer "F.Cu")
+		(net 2)
+	)
+	(segment
+		(start 115.12 128.5)
+		(end 115.12 118)
+		(width 0.2)
+		(layer "F.Cu")
+		(net 2)
+	)
+	(segment
+		(start 124 132.67)
+		(end 124 128)
+		(width 0.2)
+		(layer "F.Cu")
+		(net 2)
+	)
+	(segment
+		(start 124 128)
+		(end 115.62 128)
+		(width 0.2)
+		(layer "F.Cu")
+		(net 2)
+	)
+	(segment
+		(start 125.93 134.6)
+		(end 124 132.67)
+		(width 0.2)
+		(layer "F.Cu")
+		(net 2)
+	)
+	(segment
+		(start 115.62 128)
+		(end 115.12 128.5)
+		(width 0.2)
+		(layer "F.Cu")
+		(net 2)
+	)
+	(segment
+		(start 115.12 133.41)
+		(end 115.12 128.5)
+		(width 0.2)
+		(layer "F.Cu")
+		(net 2)
 	)
 	(segment
@@
 	)
 	(segment
+		(start 110.948 126.402)
+		(end 110.948 134.118)
+		(width 0.2)
+		(layer "B.Cu")
+		(net 5)
+	)
+	(segment
+		(start 111.75 125.6)
+		(end 110.948 126.402)
+		(width 0.2)
+		(layer "B.Cu")
+		(net 5)
+	)
+	(segment
+		(start 110.948 134.118)
+		(end 111.43 134.6)
+		(width 0.2)
+		(layer "B.Cu")
+		(net 5)
+	)
+	(segment
 		(start 111.75 91.66)
 		(end 111.25 91.16)
@@
 	)
 	(segment
+		(start 126.5 97.254816)
+		(end 126.5 91.16)
+		(width 0.2)
+		(layer "F.Cu")
+		(net 6)
+	)
+	(segment
+		(start 110.129 138.129)
+		(end 110.129 113.625816)
+		(width 0.2)
+		(layer "F.Cu")
+		(net 6)
+	)
+	(segment
+		(start 110.129 113.625816)
+		(end 126.5 97.254816)
+		(width 0.2)
+		(layer "F.Cu")
+		(net 6)
+	)
+	(segment
+		(start 111.43 139.57)
+		(end 111.5 139.5)
+		(width 0.2)
+		(layer "F.Cu")
+		(net 6)
+	)
+	(segment
+		(start 111.5 139.5)
+		(end 110.129 138.129)
+		(width 0.2)
+		(layer "F.Cu")
+		(net 6)
+	)
+	(segment
+		(start 111.43 139.6)
+		(end 111.43 139.57)
+		(width 0.2)
+		(layer "F.Cu")
+		(net 6)
+	)
+	(segment
 		(start 113.051 131.901)
 		(end 111.75 130.6)
@@
 	)
 	(segment
+		(start 126.5 88.62)
+		(end 125.399 89.721)
+		(width 0.2)
+		(layer "B.Cu")
+		(net 7)
+	)
+	(segment
+		(start 124.629 130.199)
+		(end 111.5839 130.199)
+		(width 0.2)
+		(layer "B.Cu")
+		(net 7)
+	)
+	(segment
+		(start 125.93 130.92)
+		(end 125.93 131.5)
+		(width 0.2)
+		(layer "B.Cu")
+		(net 7)
+	)
+	(segment
+		(start 111.5839 130.199)
+		(end 111.349 130.4339)
+		(width 0.2)
+		(layer "B.Cu")
+		(net 7)
+	)
+	(segment
+		(start 125.399 91.63676)
+		(end 127.551 93.78876)
+		(width 0.2)
+		(layer "B.Cu")
+		(net 7)
+	)
+	(segment
 		(start 127.551 129.299)
-		(end 127.551 93.78876)
+		(end 125.93 130.92)
 		(width 0.2)
 		(layer "B.Cu")
@@
 	(segment
 		(start 125.399 89.721)
-		(end 126.5 88.62)
-		(width 0.2)
-		(layer "B.Cu")
-		(net 7)
-	)
-	(segment
-		(start 126.25 130.6)
+		(end 125.399 91.63676)
+		(width 0.2)
+		(layer "B.Cu")
+		(net 7)
+	)
+	(segment
+		(start 127.551 93.78876)
 		(end 127.551 129.299)
 		(width 0.2)
@@
 	)
 	(segment
-		(start 127.551 93.78876)
-		(end 125.399 91.63676)
-		(width 0.2)
-		(layer "B.Cu")
-		(net 7)
-	)
-	(segment
-		(start 125.399 91.63676)
-		(end 125.399 89.721)
-		(width 0.2)
-		(layer "B.Cu")
+		(start 125.93 131.5)
+		(end 124.629 130.199)
+		(width 0.2)
+		(layer "B.Cu")
+		(net 7)
+	)
+	(segment
+		(start 111.349 130.4339)
+		(end 111.349 130.7661)
+		(width 0.2)
+		(layer "B.Cu")
+		(net 7)
+	)
+	(segment
+		(start 111.349 130.7661)
+		(end 120.1829 139.6)
+		(width 0.2)
+		(layer "B.Cu")
+		(net 7)
+	)
+	(segment
+		(start 120.1829 139.6)
+		(end 125.93 139.6)
+		(width 0.2)
+		(layer "B.Cu")

Commit message: PCB change
Routing:
- net Net-(U1-PA7_A8_D8_SCK): track 23.1 -> 31.1 mm
Changed lines of the file:
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@@
+	)
+	(segment
+		(start 121.47 115.03)
+		(end 121.5 115)
+		(width 0.2)
+		(layer "F.Cu")
+		(net 4)
+	)
+	(segment
+		(start 121.47 115.46)
+		(end 121.47 115.03)
+		(width 0.2)
+		(layer "F.Cu")
+		(net 4)
+	)
+	(segment
+		(start 121.5 115)
+		(end 121.5 107.5)
+		(width 0.2)
+		(layer "F.Cu")
+		(net 4)
 	)
 	(segment
@@
 	)
 	(segment
-		(start 126.5 88.62)
-		(end 125.399 89.721)
+		(start 125.399 89.721)
+		(end 126.5 88.62)
 		(width 0.2)
 		(layer "B.Cu")
@@
 	)
 	(segment
+		(start 125.399 103.848)
+		(end 125.399 89.721)
+		(width 0.2)
+		(layer "B.Cu")
+		(net 7)
+	)
+	(segment
 		(start 111.5839 130.199)
 		(end 111.349 130.4339)
@@
 	)
 	(segment
-		(start 125.399 91.63676)
-		(end 127.551 93.78876)
-		(width 0.2)
-		(layer "B.Cu")
-		(net 7)
-	)
-	(segment
 		(start 127.551 129.299)
 		(end 125.93 130.92)
@@
 	)
 	(segment
-		(start 125.399 89.721)
-		(end 125.399 91.63676)
-		(width 0.2)
-		(layer "B.Cu")
-		(net 7)
-	)
-	(segment
-		(start 127.551 93.78876)
+		(start 127.551 106)
 		(end 127.551 129.299)
 		(width 0.2)
@@
 		(width 0.2)
 		(layer "B.Cu")
+		(net 7)
+	)
+	(segment
+		(start 127.551 106)
+		(end 125.399 103.848)
+		(width 0.2)
+		(layer "B.Cu")

Commit message: Pcb connections
Routing:
- net Net-(U1-PA5_A9_D9_MISO): track 12.8 -> 16.9 mm
Changed lines of the file:
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@@
+	)
+	(segment
+		(start 121.47 92.38)
+		(end 121.47 96.42)
+		(width 0.2)
+		(layer "B.Cu")
+		(net 3)
 	)
 	(segment

Commit message: edits
Routing:
- net Net-(U1-PB08_A6_D6_TX): track 113.3 -> 55.8 mm
- net Net-(U1-PA9_A5_D5_SCL): track 78.7 -> 61.9 mm
- net GND: track 152.7 -> 141.2 mm
